File: support/schematics/stm32-base-board/stm32-base-board.sch (KiCad schematic (older format))
At the start: 31 parts

Commit message: Designs for a motor control board
Included layout and schematics for an SPI based bipolar stepper motor controller board using the MCP23S08 and L293Ds.
Parts:
- C1, C10, C11, C12, C2, C3, C4, C5, C6, C7, C8, C9: renamed from C?; footprint (none) -> Capacitor_Tantalum_SMD:CP_EIA-1608-08_AVX-J
- D1: renamed from D?; footprint (none) -> Diode_SMD:D_1206_3216Metric
- D2, D3: renamed from D?; footprint (none) -> LED_SMD:LED_1206_3216Metric
- FB1: renamed from FB?; footprint (none) -> Resistor_SMD:R_0805_2012Metric
- J1: renamed from J?; footprint (none) -> Connector_USB:USB_Mini-B_Lumberg_2486_01_Horizontal
- J2: renamed from J?; footprint (none) -> Connector_PinHeader_2.54mm:PinHeader_2x03_P2.54mm_Vertical
- J3: renamed from J?; footprint (none) -> Connector_PinHeader_2.54mm:PinHeader_1x04_P2.54mm_Horizontal
- R1, R2, R3, R4, R5, R6, R7, R8: renamed from R?; footprint (none) -> Resistor_SMD:R_0805_2012Metric
- SW1: renamed from SW?; footprint (none) -> Button_Switch_SMD:SW_Push_1P1T_NO_6x6mm_H9.5mm
- Y1: renamed from Y?; footprint (none) -> Crystal:Crystal_SMD_HC49-SD
- gave numbers to parts that had none: 2
