File: support/schematics/stm32-base-board/stm32-base-board.sch (KiCad schematic (older format))
At the start: 35 parts, among them J1 USB_B_Mini, J2 Boot_Pins, J3 SWDebugger, J4 Power, SW1 SW_Push, U1 AMS1117-3.3, U2 STM32F103C8Tx, Y1 8MHz

Commit message: Uploaded the schematic design for STM32 base board
Parts:
- added J5: SPI_Connector, Connector_JST:JST_EH_S4B-EH_1x04_P2.50mm_Horizontal, symbol Connector_Generic:Conn_01x04
- added J6: IR1, Connector_JST:JST_EH_S3B-EH_1x03_P2.50mm_Horizontal, symbol Connector_Generic:Conn_01x03
- added J7: IR2, Connector_JST:JST_EH_S3B-EH_1x03_P2.50mm_Horizontal, symbol Connector_Generic:Conn_01x03
- added J8: IR3, Connector_JST:JST_EH_S3B-EH_1x03_P2.50mm_Horizontal, symbol Connector_Generic:Conn_01x03
- added R10, R11, R12, R9: 20, Resistor_SMD:R_0805_2012Metric, symbol Device:R_Small
Connections:
- net labels added: IR1, IR2, IR3, MISO, MOSI, NCS, SCK
- wire segments 121 -> 146
- no-connect marks 0 -> 1
Other:
- note added: "ANALOG VOLTAGE FILTERING"
- note added: "BOOTLOADER SELECT"
- note added: "CONNECTORS"
- note added: "DECOUPLING CAPACITORS"
- note added: "EXTERNAL OSCILLATOR"
- note added: "EXTERNAL RESET CIRCUITRY"
- note added: "For SPI communication with other devices"
- note added: "For attaching a digital IR sensor"
- note added: "For external power input"
- note added: "MICROCONTROLLER"
- note added: "Note: All resistors for SPI \nare 33R"
- note added: "ROBOT BASE BOARD"
- note added: "STATUS LEDS"
- note added: "TODO:\n1/ Add MPU6050 sensor(check for SPI comm)\n2/ Add data logging capability\n3/ Maybe need more sensors"
- note added: "VOLTAGE REGULATION"
- note removed: "Analog voltage filtering"
- moved on the sheet: C1, C10, C11, C12, C13, C14, C2, C3, C4, C6, C7, C9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

Commit message: added libraries for SPI and GPIO
Parts:
- added J9: SPI_Connector, Connector_JST:JST_EH_S4B-EH_1x04_P2.50mm_Horizontal, symbol Connector_Generic:Conn_01x04
- added R13, R14, R15, R16: 20, Resistor_SMD:R_0805_2012Metric, symbol Device:R_Small
- J3: footprint Connector_PinHeader_2.54mm:PinHeader_1x04_P2.54mm_Horizontal -> Connector_PinSocket_2.54mm:PinSocket_1x04_P2.54mm_Vertical
Connections:
- net labels added: NCS2
- net labels removed: SWCLK
- wire segments 146 -> 154
Changed lines of the file:
@@
 Text GLabel 5575 5800 2    50   Input ~ 0
 SWDIO
-Text GLabel 5561 5900 2    50   Input ~ 0
-SWCLK
+Text GLabel 5510 5900 2    50   Input ~ 0
+SWDCLK
 Text GLabel 5415 6000 2    50   Input ~ 0
 PA15
@@
 F 0 "J3" H 7523 2970 50  0000 C CNN
 F 1 "SWDebugger" H 7523 3061 50  0000 C CNN
-F 2 "Connector_PinHeader_2.54mm:PinHeader_1x04_P2.54mm_Horizontal" H 7605 3395 50  0001 C CNN
+F 2 "Connector_PinSocket_2.54mm:PinSocket_1x04_P2.54mm_Vertical" H 7605 3395 50  0001 C CNN
 F 3 "~" H 7605 3395 50  0001 C CNN
 	1    7605 3395
@@
 Wire Wire Line
 	5575 5800 5415 5800
-Wire Wire Line
-	5415 5900 5561 5900
 $Comp
 L Connector_Generic:Conn_01x02 J4
@@
 For external power input
 Wire Notes Line
-	7275 3905 10875 3905
-Wire Notes Line
-	10875 3905 10875 820
-Wire Notes Line
 	10875 820  7275 820
-Wire Notes Line
-	7275 820  7275 3905
 Text Notes 7275 820  0    59   ~ 12
 CONNECTORS
-Text Notes 7280 4300 0    39   Italic 0
+Text Notes 7255 5295 0    39   Italic 0
 TODO:\n1/ Add MPU6050 sensor(check for SPI comm)\n2/ Add data logging capability\n3/ Maybe need more sensors
 Text Notes 9985 1420 0    39   Italic 0
@@
 Text Notes 7365 7525 0    98   Italic 20
 ROBOT BASE BOARD
+Wire Wire Line
+	5510 5900 5415 5900
+$Comp
+L Connector_Generic:Conn_01x04 J9
+U 1 1 5F43A4B7
+P 7605 4265
+F 0 "J9" H 7523 3840 50  0000 C CNN
+F 1 "SPI_Connector" H 7523 3931 50  0000 C CNN
+F 2 "Connector_JST:JST_EH_S4B-EH_1x04_P2.50mm_Horizontal" H 7605 4265 50  0001 C CNN
+F 3 "~" H 7605 4265 50  0001 C CNN
+	1    7605 4265
+	-1   0    0    1
+$EndComp
+Text GLabel 8155 4165 2    50   Input ~ 0
+MISO
+Text GLabel 8155 4265 2    50   Input ~ 0
+MOSI
+Text GLabel 8180 4365 2    50   Input ~ 0
+SCK
+Text GLabel 8180 4065 2    50   Input ~ 0
+NCS2
+$Comp
+L Device:R_Small R13
+U 1 1 5F43A4C1
+P 7980 4065
+F 0 "R13" V 7970 3320 50  0001 C CNN
+F 1 "20" V 7970 3495 50  0001 C CNN
+F 2 "Resistor_SMD:R_0805_2012Metric" H 7980 4065 50  0001 C CNN
+F 3 "~" H 7980 4065 50  0001 C CNN
+	1    7980 4065
+	0    1    1    0
+$EndComp
+$Comp
+L Device:R_Small R14
+U 1 1 5F43A4C7
+P 7980 4165
+F 0 "R14" V 7630 4240 50  0001 C CNN
+F 1 "20" V 7630 4340 50  0001 C CNN
+F 2 "Resistor_SMD:R_0805_2012Metric" H 7980 4165 50  0001 C CNN
+F 3 "~" H 7980 4165 50  0001 C CNN
+	1    7980 4165
+	0    1    1    0
+$EndComp
+$Comp
+L Device:R_Small R15
+U 1 1 5F43A4CD
+P 7980 4265
+F 0 "R15" V 7605 4340 50  0001 C CNN
+F 1 "20" V 7605 4440 50  0001 C CNN
+F 2 "Resistor_SMD:R_0805_2012Metric" H 7980 4265 50  0001 C CNN
+F 3 "~" H 7980 4265 50  0001 C CNN
+	1    7980 4265
+	0    1    1    0
+$EndComp
+$Comp
+L Device:R_Small R16
+U 1 1 5F43A4D3
+P 7980 4365
+F 0 "R16" V 7580 4440 50  0001 C CNN
+F 1 "20" V 7580 4540 50  0001 C CNN
+F 2 "Resistor_SMD:R_0805_2012Metric" H 7980 4365 50  0001 C CNN
+F 3 "~" H 7980 4365 50  0001 C CNN
+	1    7980 4365
+	0    1    1    0
+$EndComp
+Wire Wire Line
+	8180 4065 8080 4065
+Wire Wire Line
+	7880 4065 7805 4065
+Wire Wire Line
+	8155 4165 8080 4165
+Wire Wire Line
+	7880 4165 7805 4165
+Wire Wire Line
+	8155 4265 8080 4265
+Wire Wire Line
+	7880 4265 7805 4265
+Wire Wire Line
+	8180 4365 8080 4365
+Wire Wire Line
+	7880 4365 7805 4365
+Text Notes 7515 4525 0    50   Italic 0
+For SPI communication with other devices
+Text Notes 8425 4260 0    39   Italic 0
+Note: All resistors for SPI \nare 33R
+Wire Notes Line
+	7275 4610 10875 4610
+Wire Notes Line
+	10875 820  10875 4610
+Wire Notes Line
+	7275 820  7275 4610
 $EndSCHEMATC
