File: support/schematics/motor-controller/motor-controller.kicad_pcb (KiCad board)
At the start: 2 copper layers, 62.7 x 38.4 mm, 15 parts, among them J1 Power_Connector, J2 SPI_Connector, J3 Motor_Connector, J4 Motor_Connector, U1 AMS1117-5.0, U2 MCP23S08-xSO, U3 L293D, U4 L293D

Commit message: Updated README.md
Updated the landing README file, and added Gerber fabrication outputs for the motor controller
Routing:
- net GP4: track 37.0 -> 40.5 mm
- net M1C: track 30.3 -> 31.6 mm
- net GP5: track 44.2 -> 45.1 mm
- net M2C: track 37.9 -> 38.6 mm
